File: electronics/AutoTiller.kicad_sch (KiCad schematic)
At the start: 92 parts, among them IC1 ESP32-C3-MINI-1-N4, J1 USB_C_Receptacle_USB2.0, J3 UART, SW1 Power, SW1 Reset, SW2 +1, SW2 +15, SW2 -1, SW2 -15, SW2 L, SW2 R

Commit message: Final Rev2 PCB
Parts:
- removed C14: 2.2uF, Capacitor_SMD:C_0402_1005Metric, symbol Device:C_Small
- removed MMC5603NJ1: ~, Package_BGA:WLP-4_0.83x0.83mm_P0.4mm, symbol MMC5603NJ_Compass:MMC5603NJ
- added BT2: Battery, 18650:254 clip, symbol Device:Battery
- added C36: 0.22u, Capacitor_SMD:C_0402_1005Metric, symbol Device:C_Small
- added C37, C39: 0.1u, Capacitor_SMD:C_0402_1005Metric, symbol Device:C_Small
- added C41: 10u, Capacitor_SMD:C_0603_1608Metric, symbol Device:C_Small
- added U2: ~, Package_LGA:LGA-12_2x2mm_P0.5mm, symbol Compass:LIS2MDLTR
- BT1: footprint XT30-U:XT30-U -> 18650:254 clip
- L1: renamed from L3; footprint Inductor_SMD:L_Bourns_SRP7028A_7.3x6.6mm -> Inductor_SMD:L_Sunlord_MWSA0402S
- L2: footprint Inductor_SMD:L_Bourns_SRP7028A_7.3x6.6mm -> Inductor_SMD:L_Sunlord_MWSA0618S
- R16: renamed from R23; value 10.5k -> 6.04k
- U3: renamed from U2; footprint Connector_PinHeader_2.54mm:PinHeader_1x06_P2.54mm_Horizontal -> Connector_PinHeader_2.54mm:PinHeader_1x06_P2.54mm_Vertical
- renumbered C23 to C1, C10 to C11, C40 to C13, C12 to C14, C41 to C16, C37 to C17, C13 to C18, C42 to C19, C27 to C21, C43 to C22, C28 to C23, C29 to C24, C35 to C25, C7 to C26, C30 to C27, C36 to C28, C8 to C29, C24 to C3, C31 to C30, C39 to C31, C9 to C32, C32 to C33, C21 to C35, C5 to C38, C11 to C4, C6 to C40, C22 to C42, C25 to C5, C33 to C6, C34 to C7, C26 to C8, R22 to R10, R17 to R11, R18 to R12, R15 to R13, R19 to R14, R16 to R17, R4 to R18, R24 to R19, R27 to R2, R25 to R20, R26 to R21, R20 to R22, R21 to R23, R6 to R24, R5 to R25, R2 to R26, R28 to R3, SW1 to SW5, U3 to U1
Connections:
- net +1: now also IC1.6 (I38); no longer IC1.10 (I35)
- net +12V: no longer C38.1, C40.1, DRV8251ADDAR1.5 (VM)
- net +15: now also IC1.5 (I37); no longer IC1.9 (I34)
- net +3.3V: now also C39.1, C41.1, U2.9 (Vdd)
- net -1: now also IC1.7 (I39); no longer IC1.4 (I36)
- net -15: now also IC1.9 (I34); no longer IC1.5 (I37)
- net BC_INT: now also IC1.18 (IO13); no longer IC1.32 (IO19)
- net ENC_B: now also IC1.26 (IO10); no longer IC1.22 (IO4)
- net GND: now also SW5.2 (B), C36.2, C37.2, C39.2, C41.2, U2.11 (NC), U2.12 (NC), U2.2 (NC), U2.6 (GND), U2.8 (GND); no longer BT1.2 (-)
- net IMU_INT1: now also IC1.32 (IO19); no longer IC1.18 (IO13)
- net IMU_INT2: now also IC1.34 (IO21); no longer IC1.16 (IO14)
- net MC_IN1: now also IC1.30 (IO18); no longer IC1.29 (IO5)
- net MC_IN2: now also IC1.31 (IO23); no longer IC1.30 (IO18)
- net MC_VREF: now also IC1.29 (IO5); no longer IC1.26 (IO10)
- net QON: now also IC1.16 (IO14); no longer IC1.34 (IO21)
- net SAO: now also IC1.33 (IO22); no longer IC1.17 (IO12)
- net SCL: now also U2.1 (SCL)
- net SDA: now also U2.4 (SDA)
- net TackL: now also IC1.10 (I35); no longer IC1.6 (I38)
- net TackR: now also IC1.4 (I36); no longer IC1.7 (I39)
- net VBAT: now also BT1.1 (+), C38.1, C40.1, DRV8251ADDAR1.5 (VM); no longer SW5.1 (A)
- net Compass_INT: now reaches IC1.13 (IO25)
- net Compass_INT: now also U2.7 (INT)
- net BT2: now reaches SW5.3 (C)
- net BT2: now also BT2.2 (-)
- new net: C36.1, U2.5 (C1)
- new net BT1: BT1.2 (-), BT2.1 (+)
- new net Vdd_IO: C37.1, U2.10 (Vdd-IO), U2.3 (CS)
- no-connect marks 16 -> 15
Other:
- moved on the sheet: BT1, C35, C42, LSM6DSMTR1, SW5A

Commit message: MVP
Connections:
- net +3.3V: now also U2.3 (CS)
- net Vdd_IO: no longer names the net of C37.1, U2.10 (Vdd-IO)
- net Vdd_IO: no longer U2.3 (CS)
Other:
- moved on the sheet: C36, C37
Changed lines of the file:
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@@
     (stroke (width 0) (type default))
   )
-  (wire (pts (xy 222.25 72.39) (xy 222.25 73.66))
+  (wire (pts (xy 219.71 72.39) (xy 219.71 73.66))
     (stroke (width 0) (type default))
   )
@@
     (stroke (width 0) (type default))
   )
-  (wire (pts (xy 219.71 81.28) (xy 231.14 81.28))
+  (wire (pts (xy 212.09 81.28) (xy 231.14 81.28))
     (stroke (width 0) (type default))
   )
@@
     (stroke (width 0) (type default))
   )
-  (wire (pts (xy 222.25 67.31) (xy 240.03 67.31))
+  (wire (pts (xy 219.71 67.31) (xy 240.03 67.31))
     (stroke (width 0) (type default))
   )
@@
     (stroke (width 0) (type default))
   )
+  (wire (pts (xy 231.14 83.82) (xy 227.33 83.82))
+    (stroke (width 0) (type default))
+  )
   (wire (pts (xy 166.37 90.17) (xy 168.91 90.17))
     (stroke (width 0) (type default))
@@
     )
   )
-  (global_label "Vdd_IO" (shape input) (at 231.14 83.82 180) (fields_autoplaced)
-    (effects (font (size 1.27 1.27)) (justify right))
-    (property "Intersheetrefs" "${INTERSHEET_REFS}" (at 221.9447 83.82 0)
-      (effects (font (size 1.27 1.27)) (justify right) hide)
-    )
-  )
   (global_label "REGN" (shape input) (at 144.78 168.91 90) (fields_autoplaced)
     (effects (font (size 1.27 1.27)) (justify left))
@@
     )
   )
-  (global_label "Vdd_IO" (shape input) (at 229.87 67.31 0) (fields_autoplaced)
-    (effects (font (size 1.27 1.27)) (justify left))
-    (property "Intersheetrefs" "${INTERSHEET_REFS}" (at 239.0653 67.31 0)
-      (effects (font (size 1.27 1.27)) (justify left) hide)
-    )
-  )
   (global_label "D-" (shape input) (at 80.01 172.72 0) (fields_autoplaced)
     (effects (font (size 1.27 1.27)) (justify left))
@@
     )
   )
-  (symbol (lib_id "Device:C_Small") (at 219.71 83.82 0) (unit 1)
+  (symbol (lib_id "Device:C_Small") (at 212.09 83.82 0) (unit 1)
     (in_bom yes) (on_board yes) (dnp no)
-    (property "Reference" "C36" (at 215.9 80.01 0)
+    (property "Reference" "C36" (at 208.28 80.01 0)
       (effects (font (size 1.27 1.27)) (justify left))
     )
-    (property "Value" "0.22u" (at 212.09 82.55 0)
+    (property "Value" "0.22u" (at 204.47 82.55 0)
       (effects (font (size 1.27 1.27)) (justify left))
     )
-    (property "Footprint" "Capacitor_SMD:C_0402_1005Metric" (at 219.71 83.82 0)
+    (property "Footprint" "Capacitor_SMD:C_0402_1005Metric" (at 212.09 83.82 0)
       (effects (font (size 1.27 1.27)) hide)
     )
-    (property "Datasheet" "~" (at 219.71 83.82 0)
+    (property "Datasheet" "~" (at 212.09 83.82 0)
       (effects (font (size 1.27 1.27)) hide)
     )
@@
     )
   )
-  (symbol (lib_id "power:GND") (at 222.25 73.66 0) (unit 1)
+  (symbol (lib_id "power:GND") (at 219.71 73.66 0) (unit 1)
     (in_bom yes) (on_board yes) (dnp no) (fields_autoplaced)
-    (property "Reference" "#PWR057" (at 222.25 80.01 0)
+    (property "Reference" "#PWR057" (at 219.71 80.01 0)
       (effects (font (size 1.27 1.27)) hide)
     )
-    (property "Value" "GND" (at 222.25 78.74 0)
+    (property "Value" "GND" (at 219.71 78.74 0)
       (effects (font (size 1.27 1.27)))
     )
-    (property "Footprint" "" (at 222.25 73.66 0)
+    (property "Footprint" "" (at 219.71 73.66 0)
       (effects (font (size 1.27 1.27)) hide)
     )
-    (property "Datasheet" "" (at 222.25 73.66 0)
+    (property "Datasheet" "" (at 219.71 73.66 0)
       (effects (font (size 1.27 1.27)) hide)
     )
@@
     )
   )
-  (symbol (lib_id "power:GND") (at 219.71 86.36 0) (unit 1)
+  (symbol (lib_id "power:GND") (at 212.09 86.36 0) (unit 1)
     (in_bom yes) (on_board yes) (dnp no) (fields_autoplaced)
-    (property "Reference" "#PWR055" (at 219.71 92.71 0)
+    (property "Reference" "#PWR055" (at 212.09 92.71 0)
       (effects (font (size 1.27 1.27)) hide)
     )
-    (property "Value" "GND" (at 219.71 91.44 0)
+    (property "Value" "GND" (at 212.09 91.44 0)
       (effects (font (size 1.27 1.27)))
     )
-    (property "Footprint" "" (at 219.71 86.36 0)
+    (property "Footprint" "" (at 212.09 86.36 0)
       (effects (font (size 1.27 1.27)) hide)
     )
-    (property "Datasheet" "" (at 219.71 86.36 0)
+    (property "Datasheet" "" (at 212.09 86.36 0)
       (effects (font (size 1.27 1.27)) hide)
     )
@@
     )
   )
-  (symbol (lib_id "Device:C_Small") (at 222.25 69.85 0) (unit 1)
+  (symbol (lib_id "Device:C_Small") (at 219.71 69.85 0) (unit 1)
     (in_bom yes) (on_board yes) (dnp no) (fields_autoplaced)
-    (property "Reference" "C37" (at 224.79 69.2213 0)
+    (property "Reference" "C37" (at 222.25 69.2213 0)
       (effects (font (size 1.27 1.27)) (justify left))
     )
-    (property "Value" "0.1u" (at 224.79 71.7613 0)
+    (property "Value" "0.1u" (at 222.25 71.7613 0)
       (effects (font (size 1.27 1.27)) (justify left))
     )
-    (property "Footprint" "Capacitor_SMD:C_0402_1005Metric" (at 222.25 69.85 0)
+    (property "Footprint" "Capacitor_SMD:C_0402_1005Metric" (at 219.71 69.85 0)
       (effects (font (size 1.27 1.27)) hide)
     )
-    (property "Datasheet" "~" (at 222.25 69.85 0)
+    (property "Datasheet" "~" (at 219.71 69.85 0)
       (effects (font (size 1.27 1.27)) hide)
     )
@@
         )
       )
+    )
+  )
+  (symbol (lib_id "power:+3.3V") (at 227.33 83.82 0) (unit 1)
+    (in_bom yes) (on_board yes) (dnp no) (fields_autoplaced)
+    (property "Reference" "#PWR062" (at 227.33 87.63 0)
+      (effects (font (size 1.27 1.27)) hide)
+    )
+    (property "Value" "+3.3V" (at 227.33 80.01 0)
+      (effects (font (size 1.27 1.27)))
+    )
+    (property "Footprint" "" (at 227.33 83.82 0)
+      (effects (font (size 1.27 1.27)) hide)
+    )
+    (property "Datasheet" "" (at 227.33 83.82 0)
+      (effects (font (size 1.27 1.27)) hide)
+    )
+    (pin "1")
+    (instances
+      (project "AutoTiller"
+        (path "/8fe1d5bf-4000-444d-9640-67eaa880ff39"
+          (reference "#PWR062") (unit 1)
+        )
+      )
